File: assets/automatic_soldering_station_pcb/automatic_soldering_station_pcb.kicad_pcb (KiCad board)
At the start: 2 copper layers, 118.5 x 94.5 mm, 30 parts, among them J1 XY_MOS, J2 MAX6675, J3 MAX6675, J4 MAX6675, J5 I2C_DATA_PORT

Commit message: pcb: add pcb output files
Other:
- board text added: "APPS"
Changed lines of the file:
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@@
+		)
+	)
+	(gr_text "APPS"
+		(at 82.25 58.25 0)
+		(layer "F.SilkS")
+		(effects
+			(font
+				(face "Fira Sans Medium")
+				(size 3 3)
+				(thickness 0.3)
+				(bold yes)
+			)
+			(justify left bottom)
+		)
+		(render_cache "APPS" 0
+			(polygon
+				(pts
+					(xy 84.715265 57.74) (xy 84.12725 57.74) (xy 83.946632 57.069736) (xy 82.984926 57.069736) (xy 82.804309 57.74)
+					(xy 82.228934 57.74) (xy 82.567523 56.649699) (xy 83.094103 56.649699) (xy 83.833243 56.649699)
+					(xy 83.463764 55.256782) (xy 83.094103 56.649699) (xy 82.567523 56.649699) (xy 83.131838 54.832533)
+					(xy 83.816573 54.832533)
+				)
+			)
+			(polygon
+				(pts
+					(xy 86.062347 54.838157) (xy 86.341781 54.878061) (xy 86.566518 54.950597) (xy 86.744396 55.05128)
+					(xy 86.881943 55.17881) (xy 86.937021 55.253357) (xy 86.982922 55.335342) (xy 87.020079 55.426775)
+					(xy 87.047179 55.526058) (xy 87.064439 55.637799) (xy 87.070254 55.758152) (xy 87.067808 55.839114)
+					(xy 87.032249 56.05923) (xy 86.999467 56.15674) (xy 86.957258 56.246153) (xy 86.904846 56.329261)
+					(xy 86.843516 56.40413) (xy 86.770292 56.473778) (xy 86.688351 56.534647) (xy 86.592034 56.589993)
+					(xy 86.487075 56.635665) (xy 86.365416 56.674125) (xy 86.235333 56.701781) (xy 86.087526 56.719636)
+					(xy 85.93196 56.725537) (xy 85.591791 56.725537) (xy 85.591791 57.74) (xy 85.037482 57.74) (xy 85.037482 56.309713)
+					(xy 85.591791 56.309713) (xy 85.890012 56.309713) (xy 86.028118 56.302808) (xy 86.196625 56.266224)
+					(xy 86.319091 56.201218) (xy 86.367513 56.157247) (xy 86.408366 56.104392) (xy 86.442501 56.039407)
+					(xy 86.467793 55.963586) (xy 86.484876 55.868056) (xy 86.490666 55.758152) (xy 86.488576 55.698498)
+					(xy 86.456601 55.539841) (xy 86.427171 55.474999) (xy 86.38904 55.418577) (xy 86.340038 55.368256)
+					(xy 86.282047 55.326652) (xy 86.207488 55.290358) (xy 86.122591 55.264116) (xy 86.012594 55.245884)
+					(xy 85.890012 55.23993) (xy 85.591791 55.23993) (xy 85.591791 56.309713) (xy 85.037482 56.309713)
+					(xy 85.037482 54.832533) (xy 85.894225 54.832533)
+				)
+			)
+			(polygon
+				(pts
+					(xy 88.541901 54.838157) (xy 88.821334 54.878061) (xy 89.046072 54.950597) (xy 89.22395 55.05128)
+					(xy 89.361496 55.17881) (xy 89.416575 55.253357) (xy 89.462476 55.335342) (xy 89.499632 55.426775)
+					(xy 89.526732 55.526058) (xy 89.543992 55.637799) (xy 89.549808 55.758152) (xy 89.547361 55.839114)
+					(xy 89.511803 56.05923) (xy 89.47902 56.15674) (xy 89.436811 56.246153) (xy 89.384399 56.329261)
+					(xy 89.323069 56.40413) (xy 89.249846 56.473778) (xy 89.167904 56.534647) (xy 89.071588 56.589993)
+					(xy 88.966628 56.635665) (xy 88.844969 56.674125) (xy 88.714886 56.701781) (xy 88.567079 56.719636)
+					(xy 88.411514 56.725537) (xy 88.071345 56.725537) (xy 88.071345 57.74) (xy 87.517035 57.74) (xy 87.517035 56.309713)
+					(xy 88.071345 56.309713) (xy 88.369565 56.309713) (xy 88.507671 56.302808) (xy 88.676178 56.266224)
+					(xy 88.798644 56.201218) (xy 88.847067 56.157247) (xy 88.88792 56.104392) (xy 88.922054 56.039407)
+					(xy 88.947347 55.963586) (xy 88.964429 55.868056) (xy 88.970219 55.758152) (xy 88.968129 55.698498)
+					(xy 88.936155 55.539841) (xy 88.906724 55.474999) (xy 88.868593 55.418577) (xy 88.819592 55.368256)
+					(xy 88.7616 55.326652) (xy 88.687042 55.290358) (xy 88.602144 55.264116) (xy 88.492147 55.245884)
+					(xy 88.369565 55.23993) (xy 88.071345 55.23993) (xy 88.071345 56.309713) (xy 87.517035 56.309713)
+					(xy 87.517035 54.832533) (xy 88.373778 54.832533)
+				)
+			)
+			(polygon
+				(pts
+					(xy 90.758993 54.773914) (xy 90.627926 54.779701) (xy 90.503311 54.796763) (xy 90.387028 54.824321)
+					(xy 90.278529 54.862055) (xy 90.180563 54.908426) (xy 90.091432 54.96372) (xy 90.014009 55.02554)
+					(xy 89.946175 55.095008) (xy 89.890177 55.169268) (xy 89.844333 55.250019) (xy 89.809947 55.334689)
+					(xy 89.78628 55.424895) (xy 89.772008 55.575519) (xy 89.77792 55.684751) (xy 89.795858 55.785795)
+					(xy 89.823298 55.87213) (xy 89.861444 55.952396) (xy 89.967666 56.093217) (xy 90.123057 56.219452)
+					(xy 90.34594 56.338123) (xy 90.645603 56.447833) (xy 90.847747 56.516077) (xy 90.999336 56.584028)
+					(xy 91.077032 56.632769) (xy 91.135827 56.685082) (xy 91.172659 56.733928) (xy 91.198233 56.787458)
+					(xy 91.220567 56.914593) (xy 91.220978 56.938394) (xy 91.215227 57.013939) (xy 91.198415 57.082529)
+					(xy 91.171728 57.143115) (xy 91.135612 57.196774) (xy 91.035278 57.284381) (xy 90.895514 57.344199)
+					(xy 90.714265 57.369961) (xy 90.687552 57.370338) (xy 90.569846 57.364566) (xy 90.459019 57.347612)
+					(xy 90.254316 57.282081) (xy 90.058738 57.171927) (xy 89.939986 57.08091) (xy 89.654405 57.399647)
+					(xy 89.749344 57.484493) (xy 89.854315 57.561523) (xy 89.963237 57.626351) (xy 90.081438 57.682247)
+					(xy 90.203783 57.726651) (xy 90.334912 57.761142) (xy 90.471121 57.784418) (xy 90.615866 57.796762)
+					(xy 90.700191 57.798618) (xy 90.846796 57.79284) (xy 90.984059 57.775844) (xy 91.109425 57.748741)
+					(xy 91.225254 57.711796) (xy 91.329225 57.666516) (xy 91.423537 57.612697) (xy 91.506447 57.552025)
+					(xy 91.579583 57.483988) (xy 91.64195 57.410031) (xy 91.69434 57.329721) (xy 91.768084 57.152362)
+					(xy 91.799576 56.953197) (xy 91.800566 56.909085) (xy 91.794786 56.792831) (xy 91.77777 56.687018)
+					(xy 91.751178 56.594209) (xy 91.715029 56.509821) (xy 91.615476 56.363394) (xy 91.474744 56.237372)
+					(xy 91.279968 56.124145) (xy 91.004743 56.015836) (xy 90.93961 55.994823) (xy 90.702552 55.913946)
+					(xy 90.535013 55.838545) (xy 90.460922 55.790979) (xy 90.407291 55.740944) (xy 90.375969 55.695341)
+					(xy 90.355904 55.645623) (xy 90.343169 55.541997) (xy 90.348908 55.47633) (xy 90.365628 55.417476)
+					(xy 90.427937 55.321552) (xy 90.528841 55.250601) (xy 90.672244 55.20737) (xy 90.792698 55.198164)
+					(xy 90.905516 55.204114) (xy 91.013603 55.222314) (xy 91.111979 55.251081) (xy 91.208158 55.291589)
+					(xy 91.399724 55.411052) (xy 91.443545 55.445643) (xy 91.716669 55.130936) (xy 91.607357 55.039068)
+					(xy 91.492567 54.960222) (xy 91.386019 54.902156) (xy 91.272476 54.854594) (xy 91.156618 54.819277)
+					(xy 91.032101 54.79392)
+				)
+			)
 		)
 	)
